File: electronics/controller/axis-control.sch (KiCad schematic (older format))
At the start: 36 parts

Commit message: Update PCB design to nearly finished design.
Connections:
- net labels added: VM+, VM-
- net labels removed: +VDC, GND, VCC
- wire segments 135 -> 140
Other:
- moved on the sheet: C?, U?G, U?I
