File: electronics/controller/controller.sch (KiCad schematic (older format))
At the start: 3 parts

Commit message: Update PCB design to nearly finished design.
Parts:
- removed J? (x2): DB25, symbol bjs-connectors:DB25
- removed J?: generic-2, symbol bjs-connectors:generic-2
- added C1, C2, C3, C4, C5: 100n, Capacitor_SMD:C_0805_2012Metric_Pad1.18x1.45mm_HandSolder, symbol bjs-passives:CAPACITOR
- added J1, J8: SCREW2, wago_connectors:WAGO_MCS_MINI_02, symbol bjs-connectors:SCREW2
- added J10: TEVALULOK8W, connectors_te:VALULOK-VERT-8W, symbol bjs-connectors:TEVALULOK8W
- added J2, J3, J4: TEVALULOK12W, connectors_te:VALULOK-HCS-1-2825260-2, symbol bjs-connectors:TEVALULOK12W
- added J9: C25, symbol bjs-connectors:C25
- added LD1, LD2: LED, LED_SMD:LED_0805_2012Metric_Pad1.15x1.40mm_HandSolder, symbol bjs-discrete:LED
- added R1: RESISTOR, Resistor_SMD:R_0805_2012Metric_Pad1.20x1.40mm_HandSolder, symbol bjs-passives:RESISTOR
- added R2: 2k2, Resistor_SMD:R_0805_2012Metric_Pad1.20x1.40mm_HandSolder, symbol bjs-passives:RESISTOR
- added U1: 78L05SMD, Package_SO:SOIC-8_3.9x4.9mm_P1.27mm, symbol bjs-voltageregs:78LXXSMD
- added U2: 78L10SMD, Package_SO:SOIC-8_3.9x4.9mm_P1.27mm, symbol bjs-voltageregs:78LXXSMD
Connections:
- net labels added: +10V, +12V, 0-10V-CH1, 0-10V-CH2, GND, IN1, IN2, IN3, IN4, IN5, IN6, IN7, IN8, OUT1, OUT10, OUT11, OUT12, OUT13, OUT14, OUT15, OUT16, OUT2, OUT3, OUT4, OUT5, OUT6, OUT7, OUT8, OUT9, VCC, VDD, VSS
- wire segments 0 -> 253
Other:
- note added: "COMPUTE SIDE"
- note added: "ISOLATED POWER SUPPLY\nMACHINE SIDE"
- note added: "MACHINE SIDE"
