File: electronics/controller/filter.sch (KiCad schematic (older format))
At the start: 23 parts

Commit message: Update PCB design to nearly finished design.
Parts:
- removed C? (x2): 100n, symbol bjs-passives:CAPACITOR
- removed U?: 74AHC1G04, symbol bjs-logic:74AHC1G04
- added C?: 4u7, symbol bjs-passives:CAPACITOR
- added C? (x2): 0.1u, symbol bjs-passives:CAPACITOR
- added C? (x4): CAPACITOR, symbol bjs-passives:CAPACITOR
- added D? (x8): BAS70, symbol bjs-discrete:BAS70
- added LD? (x4): LED, symbol bjs-discrete:LED
- added O? (x4): IL217AT, symbol bjs-optocouplers:il217at
- added R? (x2): 10k, symbol bjs-passives:RESISTOR
- added R? (x12): 1K, symbol bjs-passives:RESISTOR
- added R? (x8): 10K, symbol bjs-passives:RESISTOR
- added R? (x4): RESISTOR, symbol bjs-passives:RESISTOR
- added U?: MC33204, symbol bjs-amplifiers:MC33204
- added U? (x14): 74HC14, symbol bjs-passives:74HC14
- added U?: 7810, symbol bjs-voltageregs:7810
- added U? (x4): ULN2803, symbol bjs-discrete:ULN2803
Connections:
- net labels added: +12V, INDEX, INDEX+, INDEX-, PHASEA, PHASEA+, PHASEA-, PHASEB, PHASEB+, PHASEB-, SPINDLE, SPINDLE+, SPINDLE-
- wire segments 76 -> 306
Other:
- moved on the sheet: C?, D?, O?, R?, U?A, U?B, U?C
