File: electronics/controller/controller.kicad_sch (KiCad schematic)
At the start: 17 parts, among them J1 SCREW2, J10 TEVALULOK8W, J2 TEVALULOK12W, J3 TEVALULOK12W, J4 TEVALULOK12W, J8 SCREW2, U1 78L05SMD, U2 78L10SMD

Commit message: PCB zones added and fully routed
Parts:
- removed J1, J8: SCREW2, wago_connectors:WAGO_MCS_MINI_02, symbol bjs-connectors:SCREW2
- added J1, J8: TEVALULOK4W, te-connectivity_val-u-lok_vertical:te-connectivity_val-u-lok_vertical_4_1586768-4, symbol bjs-connectors:TEVALULOK4W
Connections:
- net +12V: now also J8.1, J8.2
- net GND: now also J1.3, J1.4
- net VCC: now also J1.1, J1.2
- net VSS: now also J8.3, J8.4
Changed lines of the file:
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@@
 (kicad_sch (version 20211123) (generator eeschema)
   (paper "A4")
+  (junction (at 20.32 29.21) (diameter 0) (color 0 0 0 0)
+  )
   (junction (at 215.9 134.62) (diameter 0) (color 0 0 0 0)
   )
@@
   (junction (at 31.75 26.67) (diameter 0) (color 0 0 0 0)
   )
+  (junction (at 193.04 134.62) (diameter 0) (color 0 0 0 0)
+  )
+  (junction (at 193.04 137.16) (diameter 0) (color 0 0 0 0)
+  )
+  (junction (at 20.32 26.67) (diameter 0) (color 0 0 0 0)
+  )
   (junction (at 250.19 157.48) (diameter 0) (color 0 0 0 0)
   )
@@
     (stroke (width 0) (type default) (color 0 0 0 0))
   )
-  (wire (pts (xy 21.59 29.21) (xy 24.13 29.21))
+  (wire (pts (xy 19.05 29.21) (xy 20.32 29.21))
     (stroke (width 0) (type default) (color 0 0 0 0))
   )
@@
     (stroke (width 0) (type default) (color 0 0 0 0))
   )
+  (wire (pts (xy 20.32 29.21) (xy 24.13 29.21))
+    (stroke (width 0) (type default) (color 0 0 0 0))
+  )
   (wire (pts (xy 153.67 132.08) (xy 173.99 132.08))
     (stroke (width 0) (type default) (color 0 0 0 0))
@@
     (stroke (width 0) (type default) (color 0 0 0 0))
   )
+  (wire (pts (xy 193.04 139.7) (xy 193.04 137.16))
+    (stroke (width 0) (type default) (color 0 0 0 0))
+  )
   (wire (pts (xy 29.21 124.46) (xy 119.38 124.46))
     (stroke (width 0) (type default) (color 0 0 0 0))
@@
     (stroke (width 0) (type default) (color 0 0 0 0))
   )
+  (wire (pts (xy 19.05 31.75) (xy 20.32 31.75))
+    (stroke (width 0) (type default) (color 0 0 0 0))
+  )
   (wire (pts (xy 96.52 91.44) (xy 119.38 91.44))
     (stroke (width 0) (type default) (color 0 0 0 0))
@@
     (stroke (width 0) (type default) (color 0 0 0 0))
   )
+  (wire (pts (xy 19.05 24.13) (xy 20.32 24.13))
+    (stroke (width 0) (type default) (color 0 0 0 0))
+  )
   (wire (pts (xy 171.45 96.52) (xy 173.99 96.52))
     (stroke (width 0) (type default) (color 0 0 0 0))
@@
     (stroke (width 0) (type default) (color 0 0 0 0))
   )
+  (wire (pts (xy 20.32 31.75) (xy 20.32 29.21))
+    (stroke (width 0) (type default) (color 0 0 0 0))
+  )
   (wire (pts (xy 156.21 27.94) (xy 156.21 30.48))
     (stroke (width 0) (type default) (color 0 0 0 0))
@@
     (stroke (width 0) (type default) (color 0 0 0 0))
   )
+  (wire (pts (xy 191.77 139.7) (xy 193.04 139.7))
+    (stroke (width 0) (type default) (color 0 0 0 0))
+  )
   (wire (pts (xy 251.46 91.44) (xy 251.46 71.12))
     (stroke (width 0) (type default) (color 0 0 0 0))
@@
     (stroke (width 0) (type default) (color 0 0 0 0))
   )
+  (wire (pts (xy 193.04 137.16) (xy 198.12 137.16))
+    (stroke (width 0) (type default) (color 0 0 0 0))
+  )
   (wire (pts (xy 254 86.36) (xy 254 102.87))
     (stroke (width 0) (type default) (color 0 0 0 0))
@@
     (stroke (width 0) (type default) (color 0 0 0 0))
   )
+  (wire (pts (xy 20.32 26.67) (xy 26.67 26.67))
+    (stroke (width 0) (type default) (color 0 0 0 0))
+  )
   (wire (pts (xy 44.45 73.66) (xy 41.91 73.66))
     (stroke (width 0) (type default) (color 0 0 0 0))
@@
     (stroke (width 0) (type default) (color 0 0 0 0))
   )
+  (wire (pts (xy 20.32 24.13) (xy 20.32 26.67))
+    (stroke (width 0) (type default) (color 0 0 0 0))
+  )
   (wire (pts (xy 158.75 142.24) (xy 158.75 149.86))
     (stroke (width 0) (type default) (color 0 0 0 0))
@@
     (stroke (width 0) (type default) (color 0 0 0 0))
   )
+  (wire (pts (xy 191.77 132.08) (xy 193.04 132.08))
+    (stroke (width 0) (type default) (color 0 0 0 0))
+  )
   (wire (pts (xy 171.45 30.48) (xy 171.45 27.94))
     (stroke (width 0) (type default) (color 0 0 0 0))
   )
-  (wire (pts (xy 195.58 134.62) (xy 198.12 134.62))
+  (wire (pts (xy 191.77 134.62) (xy 193.04 134.62))
     (stroke (width 0) (type default) (color 0 0 0 0))
   )
@@
     (stroke (width 0) (type default) (color 0 0 0 0))
   )
-  (wire (pts (xy 21.59 26.67) (xy 26.67 26.67))
+  (wire (pts (xy 19.05 26.67) (xy 20.32 26.67))
+    (stroke (width 0) (type default) (color 0 0 0 0))
+  )
+  (wire (pts (xy 193.04 134.62) (xy 198.12 134.62))
+    (stroke (width 0) (type default) (color 0 0 0 0))
+  )
+  (wire (pts (xy 193.04 132.08) (xy 193.04 134.62))
     (stroke (width 0) (type default) (color 0 0 0 0))
   )
@@
     (stroke (width 0) (type default) (color 0 0 0 0))
   )
-  (wire (pts (xy 195.58 137.16) (xy 198.12 137.16))
+  (wire (pts (xy 191.77 137.16) (xy 193.04 137.16))
     (stroke (width 0) (type default) (color 0 0 0 0))
   )
@@
     )
     (pin "1")
-  )
-  (symbol (lib_id "bjs-connectors:SCREW2") (at 195.58 137.16 0) (mirror y) (unit 1)
-    (in_bom yes) (on_board yes)
-    (property "Reference" "J8" (id 0) (at 193.2432 131.445 0)
-      (effects (font (size 0.9906 0.9906)))
-    )
-    (property "Value" "SCREW2" (id 1) (at 194.31 139.7 0)
-      (effects (font (size 0.9906 0.9906)) hide)
-    )
-    (property "Footprint" "wago_connectors:WAGO_MCS_MINI_02" (id 2) (at 195.58 137.16 0)
-      (effects (font (size 0.9906 0.9906)) hide)
-    )
-    (property "Datasheet" "" (id 3) (at 195.58 137.16 0)
-      (effects (font (size 0.9906 0.9906)) hide)
-    )
-    (pin "1")
-    (pin "2")
   )
   (symbol (lib_id "bjs-discrete:LED") (at 201.93 139.7 90) (unit 1)
@@
   (symbol (lib_id "bjs-connectors:TEVALULOK12W") (at 173.99 118.11 0) (unit 1)
     (in_bom yes) (on_board yes)
-    (property "Reference" "J4" (id 0) (at 179.7812 127 0)
-      (effects (font (size 0.9906 0.9906)) (justify left))
-    )
-    (property "Value" "TEVALULOK12W" (id 1) (at 179.7812 128.905 0)
+    (property "Reference" "J4" (id 0) (at 180.34 119.38 0)
+      (effects (font (size 0.9906 0.9906)) (justify left))
+    )
+    (property "Value" "TEVALULOK12W" (id 1) (at 180.34 121.92 0)
       (effects (font (size 0.9906 0.9906)) (justify left))
     )
@@
     (pin "1")
   )
-  (symbol (lib_id "bjs-connectors:SCREW2") (at 21.59 29.21 0) (mirror y) (unit 1)
-    (in_bom yes) (on_board yes)
-    (property "Reference" "J1" (id 0) (at 19.2532 23.495 0)
-      (effects (font (size 0.9906 0.9906)))
-    )
-    (property "Value" "SCREW2" (id 1) (at 20.32 31.75 0)
-      (effects (font (size 0.9906 0.9906)) hide)
-    )
-    (property "Footprint" "wago_connectors:WAGO_MCS_MINI_02" (id 2) (at 21.59 29.21 0)
-      (effects (font (size 0.9906 0.9906)) hide)
-    )
-    (property "Datasheet" "" (id 3) (at 21.59 29.21 0)
-      (effects (font (size 0.9906 0.9906)) hide)
-    )
-    (pin "1")
-    (pin "2")
-  )
   (symbol (lib_id "power:VCC") (at 31.75 25.4 0) (unit 1)
     (in_bom yes) (on_board yes)
@@
     )
     (pin "1")
+  )
+  (symbol (lib_id "bjs-connectors:TEVALULOK4W") (at 19.05 27.94 0) (mirror y) (unit 1)
+    (in_bom yes) (on_board yes)
+    (property "Reference" "J1" (id 0) (at 15.24 19.05 0)
+      (effects (font (size 0.9906 0.9906)))
+    )
+    (property "Value" "TEVALULOK4W" (id 1) (at 19.05 21.59 0)
+      (effects (font (size 0.9906 0.9906)))
+    )
+    (property "Footprint" "te-connectivity_val-u-lok_vertical:te-connectivity_val-u-lok_vertical_4_1586768-4" (id 2) (at 19.05 27.94 0)
+      (effects (font (size 0.9906 0.9906)) hide)
+    )
+    (property "Datasheet" "" (id 3) (at 19.05 27.94 0)
+      (effects (font (size 0.9906 0.9906)) hide)
+    )
+    (pin "1")
+    (pin "2")
+    (pin "3")
+    (pin "4")
+  )
+  (symbol (lib_id "bjs-connectors:TEVALULOK4W") (at 191.77 135.89 0) (mirror y) (unit 1)
+    (in_bom yes) (on_board yes) (fields_autoplaced)
+    (property "Reference" "J8" (id 0) (at 187.96 128.4347 0)
+      (effects (font (size 0.9906 0.9906)))
+    )
+    (property "Value" "TEVALULOK4W" (id 1) (at 187.96 130.4694 0)
+      (effects (font (size 0.9906 0.9906)))
+    )
+    (property "Footprint" "te-connectivity_val-u-lok_vertical:te-connectivity_val-u-lok_vertical_4_1586768-4" (id 2) (at 191.77 135.89 0)
+      (effects (font (size 0.9906 0.9906)) hide)
+    )
+    (property "Datasheet" "" (id 3) (at 191.77 135.89 0)
+      (effects (font (size 0.9906 0.9906)) hide)
+    )
+    (pin "1")
+    (pin "2")
+    (pin "3")
+    (pin "4")
   )
   (sheet (at 119.38 24.13) (size 34.29 34.29) (fields_autoplaced)
@@
       (reference "F4") (unit 1) (value "M3") (footprint "mechanical:M3")
     )
-    (path "/00000000-0000-0000-0000-0000627c0e13"
-      (reference "J1") (unit 1) (value "SCREW2") (footprint "wago_connectors:WAGO_MCS_MINI_02")
+    (path "/66b5829a-4d44-48da-9c4b-97b33aadd48f"
+      (reference "J1") (unit 1) (value "TEVALULOK4W") (footprint "te-connectivity_val-u-lok_vertical:te-connectivity_val-u-lok_vertical_4_1586768-4")
     )
     (path "/00000000-0000-0000-0000-0000621b657b"
@@
       (reference "J4") (unit 1) (value "TEVALULOK12W") (footprint "te-connectivity_val-u-lok_vertical:te-connectivity_val-u-lok_vertical_12_1-1586768-2")
     )
-    (path "/00000000-0000-0000-0000-000061ef2953"
-      (reference "J8") (unit 1) (value "SCREW2") (footprint "wago_connectors:WAGO_MCS_MINI_02")
+    (path "/7944fd53-a48e-4b14-8f75-8d9b2da3a590"
+      (reference "J8") (unit 1) (value "TEVALULOK4W") (footprint "te-connectivity_val-u-lok_vertical:te-connectivity_val-u-lok_vertical_4_1586768-4")
     )
     (path "/00000000-0000-0000-0000-00006253f58f"
