File: electronics/controller/isolated_outputs.kicad_sch (KiCad schematic)
At the start: 44 parts, among them U4 74HC14, U5 74HC14

Commit message: Add JLCPCB fabrication output post order
Parts:
- R31, R32, R33, R34, R35, R36, R37, R38: value RESISTOR -> 330R
Changed lines of the file:
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@@
       (effects (font (size 0.9906 0.9906)))
     )
-    (property "Value" "RESISTOR" (id 1) (at 182.88 36.9316 0)
+    (property "Value" "330R" (id 1) (at 182.88 36.9316 0)
       (effects (font (size 0.9906 0.9906)))
     )
@@
       (effects (font (size 0.9906 0.9906)))
     )
-    (property "Value" "RESISTOR" (id 1) (at 182.88 52.1716 0)
+    (property "Value" "330R" (id 1) (at 182.88 52.1716 0)
       (effects (font (size 0.9906 0.9906)))
     )
@@
       (effects (font (size 0.9906 0.9906)))
     )
-    (property "Value" "RESISTOR" (id 1) (at 182.88 67.4116 0)
+    (property "Value" "330R" (id 1) (at 182.88 67.4116 0)
       (effects (font (size 0.9906 0.9906)))
     )
@@
       (effects (font (size 0.9906 0.9906)))
     )
-    (property "Value" "RESISTOR" (id 1) (at 182.88 82.6516 0)
+    (property "Value" "330R" (id 1) (at 182.88 82.6516 0)
       (effects (font (size 0.9906 0.9906)))
     )
@@
       (effects (font (size 0.9906 0.9906)))
     )
-    (property "Value" "RESISTOR" (id 1) (at 182.88 97.8916 0)
+    (property "Value" "330R" (id 1) (at 182.88 97.8916 0)
       (effects (font (size 0.9906 0.9906)))
     )
@@
       (effects (font (size 0.9906 0.9906)))
     )
-    (property "Value" "RESISTOR" (id 1) (at 182.88 113.1316 0)
+    (property "Value" "330R" (id 1) (at 182.88 113.1316 0)
       (effects (font (size 0.9906 0.9906)))
     )
@@
       (effects (font (size 0.9906 0.9906)))
     )
-    (property "Value" "RESISTOR" (id 1) (at 182.88 128.3716 0)
+    (property "Value" "330R" (id 1) (at 182.88 128.3716 0)
       (effects (font (size 0.9906 0.9906)))
     )
@@
       (effects (font (size 0.9906 0.9906)))
     )
-    (property "Value" "RESISTOR" (id 1) (at 182.88 143.6116 0)
-      (effects (font (size 0.9906 0.9906)))
-    )
+    (property "Value" "330R" (id 1) (at 182.88 143.6116 0)
+      (effects (font (size 0.9906 0.9906)))
+    )
